File: Hardware/SparkFun_Wireless_JoyStick.brd (EAGLE design)
At the start: 101.6 x 50.8 mm, 77 parts, among them J7 CORTEX_DEBUGPTH, Q1 2.5A/30V, U1 JOYSTICKPTH, U2 JOYSTICKPTH, U3 74AHC1G125, U4 AP2112K-3.3V, U5 XBEE-2B3, U6 MAX1704X, U7 MCP73831, U8 ATSAMD21G-A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

Commit message: Minor Changes
- added reset switch
- reversed power and ground on joysticks
Parts:
- added S8: (no value), SparkFun-Switches:TACTILE_SWITCH_SMD_4.6X2.8MM
Connections:
- net !RESET: now also S8.1, S8.2
- net 3.3V: now also U1.H3, U1.V3, U2.H3, U2.V3; no longer U1.H1, U1.V1, U2.H1, U2.V1
- net GND: now also S8.3, S8.4, U1.H1, U1.V1, U2.H1, U2.V1; no longer U1.H3, U1.V3, U2.H3, U2.V3
Routing:
- net !RESET: track 22.5 -> 61.7 mm, vias 1 -> 2
- net 3.3V: track 277.4 -> 272.1 mm
Other:
- board text added: "RESET"
